Commit message: .

File: aiot_ws/src/move_turtle/urdf/turtlebot3_burger.urdf (robot description, URDF)
Before this commit: robot turtlebot3_burger, 10 links, 9 joints
Joints:
- joint camera_joint: origin xyz=0.10 0.0 0.07 rpy=0 0 0 -> xyz=0.05 0.0 0.14 rpy=0 0 0
- joint flag_joint: origin xyz=0.07 0.035 0.14 rpy=0 0 0 -> xyz=0.025 -0.05 0.14 rpy=0 0 0
